File: Conc_elec/Kicad/capteur_IR/capteur_IR.sch (KiCad schematic (older format))
At the start: 3 parts, among them J1 Conn_01x03_Male, J2 Conn_01x04_Male

Commit message: avec le PCB
Parts:
- added H1, H2, H3, H4: MountingHole_Pad, MountingHole:MountingHole_3.2mm_M3_DIN965_Pad, symbol Mechanical:MountingHole_Pad
- J1: footprint (none) -> Connector_PinHeader_2.54mm:PinHeader_1x03_P2.54mm_Vertical
- J2: footprint (none) -> Connector_PinHeader_2.54mm:PinHeader_1x04_P2.54mm_Vertical
- R1: footprint (none) -> Resistor_THT:R_Axial_DIN0207_L6.3mm_D2.5mm_P10.16mm_Horizontal
Connections:
- net GND: now also H1.1, H2.1, H3.1, H4.1
Changed lines of the file:
@@
 F 0 "J1" H 2156 3228 50  0000 C CNN
 F 1 "Conn_01x03_Male" H 2156 3137 50  0000 C CNN
-F 2 "" H 2050 2950 50  0001 C CNN
+F 2 "Connector_PinHeader_2.54mm:PinHeader_1x03_P2.54mm_Vertical" H 2050 2950 50  0001 C CNN
 F 3 "~" H 2050 2950 50  0001 C CNN
 	1    2050 2950
@@
 F 0 "J2" H 2156 3978 50  0000 C CNN
 F 1 "Conn_01x04_Male" H 2156 3887 50  0000 C CNN
-F 2 "" H 2050 3700 50  0001 C CNN
+F 2 "Connector_PinHeader_2.54mm:PinHeader_1x04_P2.54mm_Vertical" H 2050 3700 50  0001 C CNN
 F 3 "~" H 2050 3700 50  0001 C CNN
 	1    2050 3700
@@
 F 0 "R1" H 2570 3696 50  0000 L CNN
 F 1 "82" H 2570 3605 50  0000 L CNN
-F 2 "" V 2430 3650 50  0001 C CNN
+F 2 "Resistor_THT:R_Axial_DIN0207_L6.3mm_D2.5mm_P10.16mm_Horizontal" V 2430 3650 50  0001 C CNN
 F 3 "~" H 2500 3650 50  0001 C CNN
 	1    2500 3650
@@
 Text Notes 1600 4250 0    50   ~ 0
 connection CNY70\nentrée: VCC, em\nsortie: rep
+$Comp
+L Mechanical:MountingHole_Pad H1
+U 1 1 5DA707C9
+P 3800 2100
+F 0 "H1" H 3900 2149 50  0000 L CNN
+F 1 "MountingHole_Pad" H 3900 2058 50  0000 L CNN
+F 2 "MountingHole:MountingHole_3.2mm_M3_DIN965_Pad" H 3800 2100 50  0001 C CNN
+F 3 "~" H 3800 2100 50  0001 C CNN
+	1    3800 2100
+	1    0    0    -1
+$EndComp
+$Comp
+L Mechanical:MountingHole_Pad H2
+U 1 1 5DA70C39
+P 4800 2100
+F 0 "H2" H 4900 2149 50  0000 L CNN
+F 1 "MountingHole_Pad" H 4900 2058 50  0000 L CNN
+F 2 "MountingHole:MountingHole_3.2mm_M3_DIN965_Pad" H 4800 2100 50  0001 C CNN
+F 3 "~" H 4800 2100 50  0001 C CNN
+	1    4800 2100
+	1    0    0    -1
+$EndComp
+$Comp
+L Mechanical:MountingHole_Pad H3
+U 1 1 5DA70EE1
+P 5750 2100
+F 0 "H3" H 5850 2149 50  0000 L CNN
+F 1 "MountingHole_Pad" H 5850 2058 50  0000 L CNN
+F 2 "MountingHole:MountingHole_3.2mm_M3_DIN965_Pad" H 5750 2100 50  0001 C CNN
+F 3 "~" H 5750 2100 50  0001 C CNN
+	1    5750 2100
+	1    0    0    -1
+$EndComp
+$Comp
+L Mechanical:MountingHole_Pad H4
+U 1 1 5DA714F5
+P 6650 2050
+F 0 "H4" H 6750 2099 50  0000 L CNN
+F 1 "MountingHole_Pad" H 6750 2008 50  0000 L CNN
+F 2 "MountingHole:MountingHole_3.2mm_M3_DIN965_Pad" H 6650 2050 50  0001 C CNN
+F 3 "~" H 6650 2050 50  0001 C CNN
+	1    6650 2050
+	1    0    0    -1
+$EndComp
+$Comp
+L capteur_IR-rescue:GND-power #PWR0101
+U 1 1 5DA71B7B
+P 3800 2300
+F 0 "#PWR0101" H 3800 2050 50  0001 C CNN
+F 1 "GND-power" H 3805 2127 50  0000 C CNN
+F 2 "" H 3800 2300 50  0001 C CNN
+F 3 "" H 3800 2300 50  0001 C CNN
+	1    3800 2300
+	1    0    0    -1
+$EndComp
+$Comp
+L capteur_IR-rescue:GND-power #PWR0102
+U 1 1 5DA71E3D
+P 4800 2300
+F 0 "#PWR0102" H 4800 2050 50  0001 C CNN
+F 1 "GND-power" H 4805 2127 50  0000 C CNN
+F 2 "" H 4800 2300 50  0001 C CNN
+F 3 "" H 4800 2300 50  0001 C CNN
+	1    4800 2300
+	1    0    0    -1
+$EndComp
+$Comp
+L capteur_IR-rescue:GND-power #PWR0103
+U 1 1 5DA7219B
+P 5750 2300
+F 0 "#PWR0103" H 5750 2050 50  0001 C CNN
+F 1 "GND-power" H 5755 2127 50  0000 C CNN
+F 2 "" H 5750 2300 50  0001 C CNN
+F 3 "" H 5750 2300 50  0001 C CNN
+	1    5750 2300
+	1    0    0    -1
+$EndComp
+$Comp
+L capteur_IR-rescue:GND-power #PWR0104
+U 1 1 5DA723E2
+P 6650 2300
+F 0 "#PWR0104" H 6650 2050 50  0001 C CNN
+F 1 "GND-power" H 6655 2127 50  0000 C CNN
+F 2 "" H 6650 2300 50  0001 C CNN
+F 3 "" H 6650 2300 50  0001 C CNN
+	1    6650 2300
+	1    0    0    -1
+$EndComp
+Wire Wire Line
+	3800 2200 3800 2300
+Wire Wire Line
+	4800 2200 4800 2300
+Wire Wire Line
+	5750 2200 5750 2300
+Wire Wire Line
+	6650 2150 6650 2300
 $EndSCHEMATC
