File: Conc_elec/Kicad/capteur_IR/emetteur.sch (KiCad schematic (older format))
At the start: 5 parts, among them U1 NE555

Commit message: avec le PCB
Parts:
- C1, C2: footprint (none) -> Capacitor_THT:C_Rect_L7.0mm_W2.5mm_P5.00mm
- R2, R3: footprint (none) -> Resistor_THT:R_Axial_DIN0207_L6.3mm_D2.5mm_P10.16mm_Horizontal
- U1: footprint (none) -> Package_DIP:DIP-8_W7.62mm
Changed lines of the file:
@@
 F 0 "U1" H 4250 4228 50  0000 C CNN
 F 1 "NE555" H 4250 4137 50  0000 C CNN
-F 2 "" H 4250 3650 50  0001 C CNN
+F 2 "Package_DIP:DIP-8_W7.62mm" H 4250 3650 50  0001 C CNN
 F 3 "http://www.ti.com/lit/ds/symlink/ne555.pdf" H 4250 3650 50  0001 C CNN
 	1    4250 3650
@@
 F 0 "C2" H 3815 4196 50  0000 L CNN
 F 1 "100n" H 3815 4105 50  0000 L CNN
-F 2 "" H 3738 4000 50  0001 C CNN
+F 2 "Capacitor_THT:C_Rect_L7.0mm_W2.5mm_P5.00mm" H 3738 4000 50  0001 C CNN
 F 3 "~" H 3700 4150 50  0001 C CNN
 	1    3700 4150
@@
 F 0 "C1" H 3565 4796 50  0000 L CNN
 F 1 "10n" H 3565 4705 50  0000 L CNN
-F 2 "" H 3488 4600 50  0001 C CNN
+F 2 "Capacitor_THT:C_Rect_L7.0mm_W2.5mm_P5.00mm" H 3488 4600 50  0001 C CNN
 F 3 "~" H 3450 4750 50  0001 C CNN
 	1    3450 4750
@@
 F 0 "R2" H 5070 4246 50  0000 L CNN
 F 1 "6.8k" H 5070 4155 50  0000 L CNN
-F 2 "" V 4930 4200 50  0001 C CNN
+F 2 "Resistor_THT:R_Axial_DIN0207_L6.3mm_D2.5mm_P10.16mm_Horizontal" V 4930 4200 50  0001 C CNN
 F 3 "~" H 5000 4200 50  0001 C CNN
 	1    5000 4200
@@
 F 0 "R3" V 5043 3650 50  0000 C CNN
 F 1 "2.7k" V 5134 3650 50  0000 C CNN
-F 2 "" V 5180 3650 50  0001 C CNN
+F 2 "Resistor_THT:R_Axial_DIN0207_L6.3mm_D2.5mm_P10.16mm_Horizontal" V 5180 3650 50  0001 C CNN
 F 3 "~" H 5250 3650 50  0001 C CNN
 	1    5250 3650
