File: Conc_elec/Kicad/capteur_IR/recepteur.sch (KiCad schematic (older format))
At the start: 11 parts, among them U2 LM324

Commit message: avec le PCB
Parts:
- C3, C4, C5, C6: footprint (none) -> Capacitor_THT:C_Rect_L7.0mm_W2.5mm_P5.00mm
- D1: footprint (none) -> Diode_THT:D_A-405_P10.16mm_Horizontal
- R4, R5, R6, R7, R8: footprint (none) -> Resistor_THT:R_Axial_DIN0207_L6.3mm_D2.5mm_P10.16mm_Horizontal
- U2: footprint (none) -> Package_DIP:DIP-14_W7.62mm_Socket
Changed lines of the file:
@@
 F 0 "U2" H 2600 3033 50  0000 C CNN
 F 1 "LM324" H 2600 3124 50  0000 C CNN
-F 2 "" H 2550 3500 50  0001 C CNN
+F 2 "Package_DIP:DIP-14_W7.62mm_Socket" H 2550 3500 50  0001 C CNN
 F 3 "http://www.ti.com/lit/ds/symlink/lm2902-n.pdf" H 2650 3600 50  0001 C CNN
 	1    2600 3400
@@
 F 0 "U2" H 1108 4346 50  0000 L CNN
 F 1 "LM324" H 1108 4255 50  0000 L CNN
-F 2 "" H 1100 4400 50  0001 C CNN
+F 2 "Package_DIP:DIP-14_W7.62mm_Socket" H 1100 4400 50  0001 C CNN
 F 3 "http://www.ti.com/lit/ds/symlink/lm2902-n.pdf" H 1200 4500 50  0001 C CNN
 	5    1150 4300
@@
 F 0 "R4" H 1770 3546 50  0000 L CNN
 F 1 "510" H 1770 3455 50  0000 L CNN
-F 2 "" V 1630 3500 50  0001 C CNN
+F 2 "Resistor_THT:R_Axial_DIN0207_L6.3mm_D2.5mm_P10.16mm_Horizontal" V 1630 3500 50  0001 C CNN
 F 3 "~" H 1700 3500 50  0001 C CNN
 	1    1700 3500
@@
 F 0 "C3" V 1798 3300 50  0000 C CNN
 F 1 "1u" V 1889 3300 50  0000 C CNN
-F 2 "" H 2088 3150 50  0001 C CNN
+F 2 "Capacitor_THT:C_Rect_L7.0mm_W2.5mm_P5.00mm" H 2088 3150 50  0001 C CNN
 F 3 "~" H 2050 3300 50  0001 C CNN
 	1    2050 3300
@@
 F 0 "R6" V 2193 2900 50  0000 C CNN
 F 1 "33k" V 2284 2900 50  0000 C CNN
-F 2 "" V 2330 2900 50  0001 C CNN
+F 2 "Resistor_THT:R_Axial_DIN0207_L6.3mm_D2.5mm_P10.16mm_Horizontal" V 2330 2900 50  0001 C CNN
 F 3 "~" H 2400 2900 50  0001 C CNN
 	1    2400 2900
@@
 F 0 "R7" V 2593 2900 50  0000 C CNN
 F 1 "33k" V 2684 2900 50  0000 C CNN
-F 2 "" V 2730 2900 50  0001 C CNN
+F 2 "Resistor_THT:R_Axial_DIN0207_L6.3mm_D2.5mm_P10.16mm_Horizontal" V 2730 2900 50  0001 C CNN
 F 3 "~" H 2800 2900 50  0001 C CNN
 	1    2800 2900
@@
 F 0 "C4" V 2348 2600 50  0000 C CNN
 F 1 "1n" V 2439 2600 50  0000 C CNN
-F 2 "" H 2638 2450 50  0001 C CNN
+F 2 "Capacitor_THT:C_Rect_L7.0mm_W2.5mm_P5.00mm" H 2638 2450 50  0001 C CNN
 F 3 "~" H 2600 2600 50  0001 C CNN
 	1    2600 2600
@@
 F 0 "R5" H 2320 3746 50  0000 L CNN
 F 1 "1k" H 2320 3655 50  0000 L CNN
-F 2 "" V 2180 3700 50  0001 C CNN
+F 2 "Resistor_THT:R_Axial_DIN0207_L6.3mm_D2.5mm_P10.16mm_Horizontal" V 2180 3700 50  0001 C CNN
 F 3 "~" H 2250 3700 50  0001 C CNN
 	1    2250 3700
@@
 F 0 "C5" H 2715 3796 50  0000 L CNN
 F 1 "1u" H 2715 3705 50  0000 L CNN
-F 2 "" H 2638 3600 50  0001 C CNN
+F 2 "Capacitor_THT:C_Rect_L7.0mm_W2.5mm_P5.00mm" H 2638 3600 50  0001 C CNN
 F 3 "~" H 2600 3750 50  0001 C CNN
 	1    2600 3750
@@
 F 0 "D1" H 3150 3184 50  0000 C CNN
 F 1 "D" H 3150 3275 50  0000 C CNN
-F 2 "" H 3150 3400 50  0001 C CNN
+F 2 "Diode_THT:D_A-405_P10.16mm_Horizontal" H 3150 3400 50  0001 C CNN
 F 3 "~" H 3150 3400 50  0001 C CNN
 	1    3150 3400
@@
 F 0 "C6" H 3515 3696 50  0000 L CNN
 F 1 "10n" H 3515 3605 50  0000 L CNN
-F 2 "" H 3438 3500 50  0001 C CNN
+F 2 "Capacitor_THT:C_Rect_L7.0mm_W2.5mm_P5.00mm" H 3438 3500 50  0001 C CNN
 F 3 "~" H 3400 3650 50  0001 C CNN
 	1    3400 3650
@@
 F 0 "R8" H 3770 3696 50  0000 L CNN
 F 1 "39k" H 3770 3605 50  0000 L CNN
-F 2 "" V 3630 3650 50  0001 C CNN
+F 2 "Resistor_THT:R_Axial_DIN0207_L6.3mm_D2.5mm_P10.16mm_Horizontal" V 3630 3650 50  0001 C CNN
 F 3 "~" H 3700 3650 50  0001 C CNN
 	1    3700 3650
